File: CYCLOPS.kicad_sch (KiCad schematic)
At the start: 71 parts, among them J1 XT60, J2 B4B-XH-A, SW1 SPST, U1 TMC2209, U2 RP2350 Pico 2, U3 LMR33630ADDA, U4 TPS259470ARPWR, U5 LMR33630ADDA, U6 MLX90316KDC-BCG-000-RE, U7 LSM6DSRXTR

Commit message: commit
Parts:
- removed C26: 100uF, Capacitor_SMD:C_0805_2012Metric, symbol Device:C_Small
- removed D1: SMBJ18CA, easyeda2kicad:SMB_L4.6-W3.6-LS5.3-BI, symbol easyeda2kicad:SMBJ18CA_C83327
- added C28, C32, C35, C36, C40, C48: 100nF, Capacitor_SMD:C_0805_2012Metric, symbol Device:C_Small
- added C30, C39: 330uF, Capacitor_THT:CP_Radial_D10.0mm_P5.00mm_P7.50mm, symbol Device:C_Polarized_Small_US
- added C33: 100uF, Capacitor_SMD:C_0805_2012Metric, symbol Device:C_Small
- added C34: 100uF, symbol Device:C_Polarized_Small
- added C37: 2.2uF, Capacitor_SMD:C_0805_2012Metric, symbol Device:C_Small
- added C38: 22nF, Capacitor_SMD:C_0805_2012Metric, symbol Device:C_Small
- added C41, C42: 10uF, Capacitor_SMD:C_2220_5750Metric, symbol Device:C_Small
- added C43, C44, C45, C46: 470pF, Capacitor_SMD:C_0805_2012Metric, symbol Device:C_Small
- added C47: 1uF, Capacitor_SMD:C_2220_5750Metric, symbol Device:C_Small
- added D11: SMB28A, easyeda2kicad:SMB_L4.6-W3.6-LS5.3-RD, symbol easyeda2kicad:SMBJ17A
- added D12: SMBJ15A, easyeda2kicad:SMB_L4.6-W3.6-LS5.3-RD, symbol easyeda2kicad:SMBJ17A
- added D2: SMBJ17A, easyeda2kicad:SMB_L4.6-W3.6-LS5.3-RD, symbol easyeda2kicad:SMBJ17A
- added D9: LED_WHITE, LED_SMD:LED_0805_2012Metric, symbol Device:LED_Small
- added J3, J4: B4B-XH-A, easyeda2kicad:CONN-TH_B4B-XH-A-LF-SN, symbol easyeda2kicad:B4B-XH-A
- added JP1: Open, symbol Jumper:Jumper_2_Small_Open
- added Q1: 2N7002, Package_TO_SOT_SMD:SOT-23, symbol Transistor_FET:2N7002
- added R10: 1k, Resistor_SMD:R_0805_2012Metric, symbol Device:R_Small
- added R18: 1.1k, Resistor_SMD:R_0805_2012Metric, symbol Device:R_Small
- added R19, R20: 470m, Resistor_SMD:R_1206_3216Metric, symbol Device:R_Small
- added R21: 220, Resistor_SMD:R_0805_2012Metric, symbol Device:R_Small
- added TP11, TP5, TP6, TP7, TP8, TP9: TestPoint_Small, TestPoint:TestPoint_Pad_3.0x3.0mm, symbol Connector:TestPoint_Small
- C1: renamed from C7; Dielectric (none) -> X7R
- C10: renamed from C8; V Rating (none) -> 10V
- C11: renamed from C18; V Rating (none) -> 10V
- C2: renamed from C15; Dielectric (none) -> X7R
- C27: V Rating 50V -> (none)
- C3: renamed from C6; Dielectric (none) -> X7R
- C4: renamed from C16; Dielectric (none) -> X7R
- C5: renamed from C10; V Rating (none) -> 16V
- C7: renamed from C17; V Rating (none) -> 16V
- F1: renamed from F2; LCSC Part C151092 -> C178940; MPN 0297003.WXNV -> 0297004.WXNV
- U3: renamed from U6; value MLX90316KDC-BCG-000-RE -> MLX90316xDC-BDG-100-RE
- renumbered C1 to C12, C9 to C13, C2 to C14, C19 to C15, C11 to C16, C20 to C17, C30 to C18, C12 to C19, C21 to C20, C13 to C21, C14 to C23, C23 to C24, C3 to C26, C24 to C29, C28 to C31, C4 to C6, C5 to C8, C31 to C9, D8 to D1, D9 to D3, D10 to D4, D11 to D5, D2 to D6, D3 to D7, D4 to D8, R13 to R1, R14 to R11, R5 to R12, R11 to R13, R6 to R14, R12 to R15, R15 to R16, R16 to R17, R1 to R2, R2 to R3, R3 to R4, R7 to R5, R8 to R6, R9 to R7, R10 to R8, R4 to R9, TP3 to TP1, TP1 to TP2, TP2 to TP3, U3 to U1, U5 to U2, U1 to U5, U2 to U6
Connections:
- net GND: now also C27.2, U5.18 (GND), U5.29 (EP), U5.3 (GND), C28.2, C32.2, C33.2, C34.2, C35.2, C36.2, C37.2, C43.2, C44.2, C45.2, C46.2, D12.2 (A), D2.2 (A), D9.1 (K), Q1.2 (S), R19.2, R20.2; no longer U6.3 (GND), U6.38 (GND)
- net VBAT_PROT: now also D8.1 (C), C32.1, C33.1, C34.1
- net VBAT_SENSE: now also U6.31 (GPIO26_ADC0)
- net at C6.1, F1.2, R1.2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: now also D2.1 (C)
- net OB2: now reaches U5.1 (OB2)
- net OB2: now also C46.1, TP8.1
- net DIAG: now reaches U5.11 (DIAG)
- net DIAG: now also R21.1
- net INDEX: now reaches U5.12 (INDEX)
- net OA2: now reaches U5.21 (OA2)
- net OA2: now also C44.1, TP5.1
- net at U5.22 (VS): now also U5.28 (VS), C30.1, C39.1, C40.1, C41.1, C42.1, C47.1, C48.1, D11.1 (C)
- net BRA: now reaches U5.23 (BRA)
- net BRA: now also C36.1, R19.1, TP9.1
- net OA1: now reaches U5.24 (OA1)
- net OA1: now also C43.1, TP6.1
- net OB1: now reaches U5.26 (OB1)
- net OB1: now also C45.1, TP7.1
- net BRB: now reaches U5.27 (BRB)
- net BRB: now also C35.1, R20.1, TP11.1
- net at U5.4 (CPO): now also C38.2
- net at U5.5 (CPI): now also C38.1
- net at U5.6 (VCP): now also C48.2
- net at U5.8 (5VOUT): now also C37.1, D12.1 (C), JP1.2 (B)
- net IMU_SDO: now reaches U6.11 (GPIO8)
- net IMU_CS: now reaches U6.12 (GPIO9)
- net IMU_CS: now also U7.12 (CS)
- net IMU_SCL: now reaches U6.14 (GPIO10)
- net IMU_SCL: now also U7.13 (SCL)
- net IMU_SDA: now reaches U6.15 (GPIO11)
- net IMU_SDA: now also U7.14 (SDA)
- net IMU_INT1: now reaches U6.16 (GPIO12)
- net IMU_INT2: now reaches U6.17 (GPIO13)
- net IMU_INT2: now also U7.9 (INT2)
- net ENCODER_CS: now reaches U6.22 (GPIO17)
- net ENCODER_CS: now also U3.3 (~{SS}/Switch)
- net ENCODER_SCK: now reaches U6.24 (GPIO18)
- net ENCODER_SCK: now also U3.4 (OUT2/SCLK)
- net at U6.25 (GPIO19): now also Q1.1 (G)
- net ENCODER_OUT: now reaches U6.26 (GPIO20)
- net ENCODER_OUT: now also U3.5 (OUT/MOSI/MISO), Q1.3 (D), R10.1
- net PICO_3V3: now reaches U6.36 (3V3)
- net PICO_3V3: now also U7.8 (Vdd), C28.1, R10.2
- new net: C30.2, C39.2, C40.2, C41.2, C42.2, D11.2 (A), R18.2
- new net: C47.2, R18.1
- new net: D9.2 (A), R21.2
- new net +VM: JP1.1 (A)
- no-connect marks 2 -> 5
Other:
- note added: "Accelerometer / IMU"
- note added: "RPi Pico 2"
- note added: "Rotary Position Encoder"
- moved on the sheet: C18, C25, C29, C3, C31, C4, C9, D7, D8, J2, U3, U6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
